Commit message: project 2

File: catkin_ws/src/my_robot/urdf/my_robot.xacro (robot description, xacro)
@@ -22,5 +22,5 @@
       <origin xyz="0 0 0" rpy=" 0 0 0"/>
       <geometry>
-        <box size=".4 .2 .1"/>
+        <box size=".5 .3 .1"/>
       </geometry>
     </collision>
@@ -28,5 +28,5 @@
       <origin xyz="0 0 0" rpy=" 0 0 0"/>
       <geometry>
-        <box size=".4 .2 .1"/>
+        <box size=".5 .3 .1"/>
       </geometry>
     </visual>
@@ -56,4 +56,42 @@
     </visual>
   </link>
+<link name='left_wheel'>
+  <visual>
+    <origin xyz="0 0 0" rpy="0 1.5707 1.5707"/>
+    <geometry>
+      <cylinder radius="0.12" length="0.055"/>
+    </geometry>
+  </visual>
+  <collision>
+    <origin xyz="0 0 0" rpy="0 1.5707 1.5707"/>
+    <geometry>
+    <cylinder radius="0.12" length="0.055"/>
+    </geometry>
+  </collision>
+  <inertial>
+    <mass value="5.0"/>
+    <origin xyz="0 0 0" rpy="0 1.5707 1.5707"/>
+    <inertia ixx="0.1" ixy="0" ixz="0" iyy="0.1" iyz="0" izz="0.1"/>
+  </inertial>
+</link>
+<link name='right_wheel'>
+  <visual>
+    <origin xyz="0 0 0" rpy="0 1.5707 1.5707"/>
+    <geometry>
+      <cylinder radius="0.12" length="0.055"/>
+    </geometry>
+  </visual>
+  <collision>
+    <origin xyz="0 0 0" rpy="0 1.5707 1.5707"/>
+    <geometry>
+    <cylinder radius="0.12" length="0.055"/>
+    </geometry>
+  </collision>
+  <inertial>
+    <mass value="5.0"/>
+    <origin xyz="0 0 0" rpy="0 1.5707 1.5707"/>
+    <inertia ixx="0.1" ixy="0" ixz="0" iyy="0.1" iyz="0" izz="0.1"/>
+  </inertial>
+</link>
   <joint type="continuous" name="left_wheel_hinge">
     <origin xyz="0 0.15 0" rpy="0 0 0"/>
@@ -65,5 +103,5 @@
   </joint>
    <joint type="continuous" name="right_wheel_hinge">
-    <origin xyz="0 0.15 0" rpy="0 0 0"/>
+    <origin xyz="0 -0.15 0" rpy="0 0 0"/>
     <child link="right_wheel"/>
     <parent link="chassis"/>
@@ -73,12 +111,16 @@
   </joint>
   <link name='camera'>
-    <origin xyz= "0,0,0,0,0,0"/>
-    <geometry>
-      <box size=".05 .05 .05"/>
-    </geometry>
-    <mass"0.1"/>
-    <box_inertia m="0.1" x="0.05" y="0.05" z="0.05" />
-    <intertia ixx="1e-6" ixy="0" ixz="0" iyy="1e-6" iyz="0" izz="1e-6"/>
- </link>
+    <origin xyz="0 0 0" rpy = "0 0 0"/>
+    <visual>
+	<geometry>
+          <box size=".05 .05 .05"/>
+	</geometry>
+    </visual>
+    <intertial>
+      <mass value ="0.1"/>
+     <box_inertia m="0.1" x="0.05" y="0.05" z="0.05" />
+     <intertia ixx="1e-6" ixy="0" ixz="0" iyy="1e-6" iyz="0" izz="1e-6"/>
+   </intertial>
+  </link>
  <joint type="fixed" name="camera_joint">
     <origin xyz="0.2 0 0" rpy="0 0 0"/>
@@ -88,28 +130,38 @@
   </joint>
   <link name='hokuyo'>
-    <origin xyz= "0,0,0,0,0,0"/>
-    <geometry>
-      <box size=".01 .01 .1"/>
-    </geometry>
-    <collision name='collision'>
-      <origin xyz="0 0 0" rpy=" 0 0 0"/>
+    <collision>
+      <origin xyz="0 0 0" rpy="0 0 0"/>
       <geometry>
         <box size=".1 .1 .1"/>
       </geometry>
     </collision>
-    <visual name='hokuyo_visual'>
+    <visual>
       <origin xyz="0 0 0" rpy=" 0 0 0"/>
       <geometry>
-        “package://my_robot/meshes/hokuyo.dae”
+        <mesh filename="package://my_robot/meshes/hokuyo.dae"/>
       </geometry>
     </visual>
-    <mass"1e-5"/>
-    <intertia ixx="1e-6" ixy="0" ixz="0" iyy="1e-6" iyz="0" izz="1e-6"/>
+    <intertial>
+      <mass value ="1e-5"/>
+      <intertia ixx="1e-6" ixy="0" ixz="0" iyy="1e-6" iyz="0" izz="1e-6"/>
+    </intertial>
  </link>
  <joint type="fixed" name="hokuyo_joint">
-    <origin xyz="0.15 0.1 0" rpy="0 0 0"/>
+    <origin xyz="0.15 0 0.1" rpy="0 0 0"/>
     <child link="hokuyo"/>
     <parent link="chassis"/>
     <axis xyz="0 1 0" rpy="0 0 0"/>
   </joint>
+  <gazebo reference="chassis">
+    <material>Gazebo/Blue</material>
+  </gazebo>
+  <gazebo reference="left_wheel">
+    <material>Gazebo/Orange</material>
+  </gazebo>
+  <gazebo reference="right_wheel">
+    <material>Gazebo/Orange</material>
+  </gazebo>
+ <gazebo reference="camera">
+    <material>Gazebo/Purple</material>
+  </gazebo>
 </robot>
